File: ml_multigate.kicad_pcb (KiCad board)
At the start: 2 copper layers, 171 x 101 mm, 2 parts, among them U1 4001, U2 4001

Commit message: Update ml_multigate.kicad_pcb
Parts:
- removed U1: 4001, Package_DIP:DIP-14_W7.62mm

Commit message: Update ml_multigate.kicad_pcb
Parts:
- removed U2: 4001, Package_DIP:DIP-14_W7.62mm
